Commit message: Dual robot calibration and set-up

File: 2_dual_robot/2_docker/set-up/abb_irb2600_12_185_dual_config/config/gazebo_mid_robot_dual_cell.urdf (robot description, URDF)
Before this commit: robot mid_robot_dual_cell, 21 links, 20 joints
Joints:
- joint robotB_joint: origin xyz=2.5 0 0 rpy=-0 0 -3.1415926 -> xyz=3.070587026068542 0.019064029578026894 0.015637209791168258 rpy=0.00041166767187156717 0.005882192447675842 -3.129394251246824

File: 2_dual_robot/2_docker/set-up/abb_irb2600_12_185_dual_support/urdf/abb_irb2600_dual.xacro (robot description, xacro)
@@ -13,5 +13,5 @@
     <parent link="world" />
     <child link = "robotB_base_link" />
-    <origin xyz="2.5	0	0" rpy="-0	0	-3.1415926"/>
+    <origin xyz="3.070587026068542	0.019064029578026894	0.015637209791168258" rpy="0.00041166767187156717	0.005882192447675842	-3.129394251246824"/>
   </joint>
 </robot>
