Commit message: Moved the robot on 240814, update for new calibration

File: 2_dual_robot/2_docker/for-use/abb_irb2600_12_185_dual_config/config/gazebo_mid_robot_dual_cell.urdf (robot description, URDF)
Before this commit: robot mid_robot_dual_cell, 21 links, 20 joints
Joints:
- joint robotB_joint: origin xyz=3.070587026068542 0.019064029578026894 0.015637209791168258 rpy=0.00041166767187156717 0.005882192447675842 -3.129394251246824 -> xyz=2.36007471 -0.0359336150 0.000872916796  rpy=0.00185601007 0.00214706491 3.13677599

File: 2_dual_robot/2_docker/for-use/abb_irb2600_12_185_dual_config/urdf/abb_irb2600_dual.xacro (robot description, xacro)
@@ -13,5 +13,5 @@
     <parent link="world" />
     <child link = "robotB_base_link" />
-    <origin xyz="3.070587026068542	0.019064029578026894	0.015637209791168258" rpy="0.00041166767187156717	0.005882192447675842	-3.129394251246824"/>
+    <origin xyz="2.36007471	-0.0359336150	0.000872916796 " rpy="0.00185601007	0.00214706491	3.13677599"/>
   </joint>
 </robot>

File: 2_dual_robot/2_docker/set-up/abb_irb2600_12_185_dual_config/config/gazebo_mid_robot_dual_cell.urdf (robot description, URDF)
Before this commit: robot mid_robot_dual_cell, 21 links, 20 joints
Joints:
- joint robotB_joint: origin xyz=3.070587026068542 0.019064029578026894 0.015637209791168258 rpy=0.00041166767187156717 0.005882192447675842 -3.129394251246824 -> xyz=2.36007471 -0.0359336150 0.000872916796  rpy=0.00185601007 0.00214706491 3.13677599

File: 2_dual_robot/2_docker/set-up/abb_irb2600_12_185_dual_support/urdf/abb_irb2600_dual.xacro (robot description, xacro)
@@ -13,5 +13,5 @@
     <parent link="world" />
     <child link = "robotB_base_link" />
-    <origin xyz="3.070587026068542	0.019064029578026894	0.015637209791168258" rpy="0.00041166767187156717	0.005882192447675842	-3.129394251246824"/>
+    <origin xyz="2.36007471	-0.0359336150	0.000872916796 " rpy="0.00185601007	0.00214706491	3.13677599"/>
   </joint>
 </robot>
